File: picopico.kicad_pcb (KiCad board)
At the start: 2 copper layers, 0 parts

Commit message: rev1
Parts:
- added C1: CL05B104KO5NNNC, JLC2KiCadLib:C0402, F.Cu at (60.4, 54.2)
- added C10: CL05A105KA5NQNC, JLC2KiCadLib:C0402, F.Cu at (60.4, 50.7)
- added C11: CL05B104KO5NNNC, JLC2KiCadLib:C0402, F.Cu at (62.6, 50.7)
- added C12: CL05B104KO5NNNC, JLC2KiCadLib:C0402, F.Cu at (64.7, 50.7)
- added C13: CL05A105KA5NQNC, JLC2KiCadLib:C0402, F.Cu at (66.9, 50.7)
- added C14: CL05B104KO5NNNC, JLC2KiCadLib:C0402, F.Cu at (63.5, 59.2)
- added C15: CL05B104KO5NNNC, JLC2KiCadLib:C0402, F.Cu at (63.5, 57.1)
- added C16: CL05B104KO5NNNC, JLC2KiCadLib:C0402, F.Cu at (60.4, 47.2)
- added C17: CL05B104KO5NNNC, JLC2KiCadLib:C0402, F.Cu at (62.6, 47.2)
- added C18: CL05B104KO5NNNC, JLC2KiCadLib:C0402, F.Cu at (64.7, 47.2)
- added C19: CL05B104KO5NNNC, JLC2KiCadLib:C0402, F.Cu at (66.9, 47.2)
- added C2: CL10A106KP8NNNC, JLC2KiCadLib:C0603, F.Cu at (70.7, 41.4)
- added C3: CL10C220JB8NNNC, JLC2KiCadLib:C0603, F.Cu at (73.4, 41.4)
- added C4: CL10A106KP8NNNC, JLC2KiCadLib:C0603, F.Cu at (76.1, 41.4)
- added C5: CL05B104KO5NNNC, JLC2KiCadLib:C0402, F.Cu at (62.6, 54.2)
- added C6: CL05B104KO5NNNC, JLC2KiCadLib:C0402, F.Cu at (64.7, 54.2)
- added C7: CL05A106MQ5NUNC, JLC2KiCadLib:C0402, F.Cu at (66.9, 54.2)
- added C8: 0402CG220J500NT, JLC2KiCadLib:C0402, F.Cu at (66.9, 59.2)
- added C9: 0402CG220J500NT, JLC2KiCadLib:C0402, F.Cu at (66.9, 57.1)
- added D1: WS2812B, LED_SMD:LED_WS2812B_PLCC4_5.0x5.0mm_P3.2mm, F.Cu at (28.0, 19.3)
- added D2: LED, LED_SMD:LED_0402_1005Metric, F.Cu at (77.5, 22.8)
- added D3: 0402ESDA-05N, JLC2KiCadLib:D0402-BI, B.Cu at (91.7, 107.4)
- added D4: 0402ESDA-05N, JLC2KiCadLib:D0402-BI, B.Cu at (89.5, 107.4)
- added D5: 0402ESDA-05N, JLC2KiCadLib:D0402-BI, B.Cu at (87.4, 107.4)
- added D6: 0402ESDA-05N, JLC2KiCadLib:D0402-BI, B.Cu at (85.2, 107.4)
- added F1: nSMD050-24V, JLC2KiCadLib:F1206, F.Cu at (63.7, 43.8)
- added FLASH1: W25Q16JVUXIQ, JLC2KiCadLib:USON-8_L3.0-W2.0-P0.50-BL-EP, F.Cu at (64.2, 40.9)
- added G2: LOGO, zeriparrot:zeriparrot, F.Cu at (73.5, 99.9)
- added H1: MountingHole, MountingHole:MountingHole_2.2mm_M2, F.Cu at (18.9, 18.9)
- added H10: Switch_Hole, BrownSugar_KBD:Switch_Hole, F.Cu at (50.8, 84.7)
- added H11: Switch_Hole, BrownSugar_KBD:Switch_Hole, F.Cu at (31.7, 103.9)
- added H12: RotaryEncoder_EC11-Hole, BrownSugar_KBD:RotaryEncoder_EC11-Hole, F.Cu at (51.3, 103.9)
- added H2: MountingHole, MountingHole:MountingHole_2.2mm_M2, F.Cu at (102.2, 18.9)
- added H3: MountingHole, MountingHole:MountingHole_2.2mm_M2, F.Cu at (19.1, 62.2)
- added H4: MountingHole, MountingHole:MountingHole_2.2mm_M2, F.Cu at (102.2, 62.2)
- added H5: MountingHole, MountingHole:MountingHole_2.2mm_M2, F.Cu at (19.0, 68.9)
- added H6: MountingHole, MountingHole:MountingHole_2.2mm_M2, F.Cu at (102.3, 68.9)
- added H7: MountingHole, MountingHole:MountingHole_2.2mm_M2, F.Cu at (19.1, 112.2)
- added H8: MountingHole, MountingHole:MountingHole_2.2mm_M2, F.Cu at (102.3, 112.2)
- added H9: Switch_Hole, BrownSugar_KBD:Switch_Hole, F.Cu at (31.7, 84.7)
- added J1: USB_C_Receptacle_USB2.0_14P, Connector_USB:USB_C_Receptacle_HRO_TYPE-C-31-M-12, B.Cu at (85.0, 18.9)
- added J2: USB_C_Receptacle_USB2.0_14P, Connector_USB:USB_C_Receptacle_HRO_TYPE-C-31-M-12, F.Cu at (101.6, 104.4)
- added L1: SWPA3015S2R2NT, JLC2KiCadLib:IND-SMD_L3.0-W3.0, F.Cu at (75.1, 27.5)
- added R1: 0402WGF5101TCE, JLC2KiCadLib:R0402, B.Cu at (60.4, 47.9)
- added R10: 0402WGF1002TCE, JLC2KiCadLib:R0402, B.Cu at (66.9, 50.9)
- added R11: 0402WGF1001TCE, JLC2KiCadLib:R0402, B.Cu at (63.6, 59.2)
- added R12: 0402WGF1002TCE, JLC2KiCadLib:R0402, B.Cu at (63.6, 57.0)
- added R13: 0603WAF2001T5E, JLC2KiCadLib:R0603, F.Cu at (75.4, 44.2)
- added R14: RC0402FR-0727RL, JLC2KiCadLib:R0402, B.Cu at (60.4, 53.9)
- added R15: RC0402FR-0727RL, JLC2KiCadLib:R0402, B.Cu at (62.6, 53.9)
- added R16: 0402WGF1002TCE, JLC2KiCadLib:R0402, B.Cu at (64.7, 53.9)
- added R17: 0402WGF1002TCE, JLC2KiCadLib:R0402, B.Cu at (66.9, 53.9)
- added R18: 0402WGF4701TCE, JLC2KiCadLib:R0402, B.Cu at (66.7, 59.2)
- added R19: 0402WGF5101TCE, JLC2KiCadLib:R0402, F.Cu at (92.5, 101.9)
- added R2: 0402WGF5101TCE, JLC2KiCadLib:R0402, B.Cu at (62.6, 47.9)
- added R20: 0402WGF5101TCE, JLC2KiCadLib:R0402, F.Cu at (92.6, 104.9)
- added R3: 0402WGF220JTCE, JLC2KiCadLib:R0402, B.Cu at (64.7, 47.9)
- added R4: 0402WGF5601TCE, JLC2KiCadLib:R0402, B.Cu at (66.9, 47.9)
- added R5: 0402WGF1002TCE, JLC2KiCadLib:R0402, B.Cu at (60.6, 59.2)
- added R6: 0402WGF1003TCE, JLC2KiCadLib:R0402, B.Cu at (60.6, 57.0)
- added R7: 0402WGF1503TCE, JLC2KiCadLib:R0402, B.Cu at (60.4, 50.9)
- added R8: 0402WGF6803TCE, JLC2KiCadLib:R0402, B.Cu at (62.6, 50.9)
- added R9: 0402WGF1001TCE, JLC2KiCadLib:R0402, B.Cu at (64.7, 50.9)
- added SW1: SW_PUSH, PCM_Switch_Keyboard_Hotswap_Kailh:SW_Hotswap_Kailh_MX_1.00u, F.Cu at (31.7, 33.7)
- added SW2: SW_PUSH, PCM_Switch_Keyboard_Hotswap_Kailh:SW_Hotswap_Kailh_MX_1.00u, F.Cu at (50.8, 33.7)
- added SW3: SW_PUSH, PCM_Switch_Keyboard_Hotswap_Kailh:SW_Hotswap_Kailh_MX_1.00u, F.Cu at (31.7, 52.8)
- added SW4: ~, BrownSugar_KBD:RotaryEncoder_EC11-Switch, F.Cu at (51.2, 53.4)
- added SW5: TSA343G00-250J2, JLC2KiCadLib:SW-SMD_L4.0-W2.9-LS5.0, F.Cu at (87.6, 77.3)
- added SW6: TSA343G00-250J2, JLC2KiCadLib:SW-SMD_L4.0-W2.9-LS5.0, F.Cu at (87.6, 83.7)
- added SW_BOOTSEL1: 1-1825027-7, JLC2KiCadLib:SW-TH_KH-6X6X4.3H-ZJ, B.Cu at (38.7, 19.3)
- added SW_RESET1: 1-1825027-7, JLC2KiCadLib:SW-TH_KH-6X6X4.3H-ZJ, B.Cu at (48.1, 19.3)
- added U1: 1N4002W, JLC2KiCadLib:SOD-123F_L2.8-W1.8-LS3.7-RD, F.Cu at (67.8, 41.7)
- added U10: SK6812MINI-E_C5149201, JLC2KiCadLib:LED-SMD_L3.2-W2.8-TR, B.Cu at (31.7, 38.0)
- added U11: SK6812MINI-E_C5149201, JLC2KiCadLib:LED-SMD_L3.2-W2.8-TR, B.Cu at (50.8, 38.0)
- added U12: SK6812MINI-E_C5149201, JLC2KiCadLib:LED-SMD_L3.2-W2.8-TR, B.Cu at (31.7, 57.2)
- added U13: FS-1540, JLC2KiCadLib:BUZ-SMD_5P-L15.0-W15.0-P13.7-BL, B.Cu at (77.3, 54.2)
- added U14: X1321FR-2X20-C43D24, JLC2KiCadLib:CONN-TH_40P_X1321FR-2X20-C43D24, F.Cu at (99.7, 85.7)
- added U2: TD6810, JLC2KiCadLib:SOT-23-5_L3.0-W1.7-P0.95-LS2.8-BR, F.Cu at (75.2, 37.5)
- added U3: RP2040, Package_DFN_QFN:QFN-56-1EP_7x7mm_P0.4mm_EP3.2x3.2mm, F.Cu at (66.4, 31.1)
- added U4: X1321FR-2X20-C43D24, JLC2KiCadLib:CONN-TH_40P_X1321FR-2X20-C43D24, B.Cu at (66.4, 20.1)
- added U5: 1N4148W_C81598, JLC2KiCadLib:SOD-123F_L2.7-W1.6-LS3.8-RD, B.Cu at (38.8, 42.2)
- added U6: 1N4148W_C81598, JLC2KiCadLib:SOD-123F_L2.7-W1.6-LS3.8-RD, B.Cu at (57.9, 42.2)
- added U7: 1N4148W_C81598, JLC2KiCadLib:SOD-123F_L2.7-W1.6-LS3.8-RD, B.Cu at (38.8, 61.2)
- added U8: 1N4148W_C81598, JLC2KiCadLib:SOD-123F_L2.7-W1.6-LS3.8-RD, B.Cu at (71.0, 44.7)
- added U9: BSS138, JLC2KiCadLib:SOT-23-3_L2.9-W1.3-P1.90-LS2.4-BR, B.Cu at (61.3, 62.1)
- added X1: X322512MSB4SI, JLC2KiCadLib:OSC-SMD_4P-L3.2-W2.5-BL, F.Cu at (75.3, 32.5)
- added XTRAPI_C1: 0402CG300J500NT, XTRAPI_JLC2KiCadLib:C0402, B.Cu at (89.7, 87.6)
- added XTRAPI_C10: CL05A106MQ5NUNC, XTRAPI_JLC2KiCadLib:C0402, B.Cu at (86.2, 91.9)
- added XTRAPI_C11: CL05A106MQ5NUNC, XTRAPI_JLC2KiCadLib:C0402, B.Cu at (86.2, 94.1)
- added XTRAPI_C12: CL05A106MQ5NUNC, XTRAPI_JLC2KiCadLib:C0402, B.Cu at (86.2, 96.2)
- added XTRAPI_C13: CL05A106MQ5NUNC, XTRAPI_JLC2KiCadLib:C0402, B.Cu at (86.2, 98.4)
- added XTRAPI_C14: CL31A107MQHNNNE, XTRAPI_JLC2KiCadLib:C1206, F.Cu at (87.6, 100.5)
- added XTRAPI_C15: CL05A106MQ5NUNC, XTRAPI_JLC2KiCadLib:C0402, B.Cu at (82.8, 87.6)
- added XTRAPI_C16: CL05A106MQ5NUNC, XTRAPI_JLC2KiCadLib:C0402, B.Cu at (82.8, 89.8)
- added XTRAPI_C17: CL05A106MQ5NUNC, XTRAPI_JLC2KiCadLib:C0402, B.Cu at (82.8, 91.9)
- added XTRAPI_C18: CL05A106MQ5NUNC, XTRAPI_JLC2KiCadLib:C0402, B.Cu at (82.8, 94.1)
- added XTRAPI_C2: CL05A106MQ5NUNC, XTRAPI_JLC2KiCadLib:C0402, B.Cu at (89.7, 89.8)
- added XTRAPI_C3: 0402CG300J500NT, XTRAPI_JLC2KiCadLib:C0402, B.Cu at (89.7, 91.9)
- added XTRAPI_C4: CL31A107MQHNNNE, XTRAPI_JLC2KiCadLib:C1206, F.Cu at (87.6, 104.8)
- added XTRAPI_C5: CL05A106MQ5NUNC, XTRAPI_JLC2KiCadLib:C0402, B.Cu at (89.7, 94.1)
- added XTRAPI_C6: CL05A106MQ5NUNC, XTRAPI_JLC2KiCadLib:C0402, B.Cu at (89.7, 96.2)
- added XTRAPI_C7: CL05A106MQ5NUNC, XTRAPI_JLC2KiCadLib:C0402, B.Cu at (89.7, 98.4)
- added XTRAPI_C8: CL05A106MQ5NUNC, XTRAPI_JLC2KiCadLib:C0402, B.Cu at (86.2, 87.6)
- added XTRAPI_C9: CL05A106MQ5NUNC, XTRAPI_JLC2KiCadLib:C0402, B.Cu at (86.2, 89.8)
- added XTRAPI_R2: 0402WGF1002TCE, XTRAPI_JLC2KiCadLib:R0402, B.Cu at (94.3, 103.2)
- added XTRAPI_R4: 0402WGF1001TCE, XTRAPI_JLC2KiCadLib:R0402, B.Cu at (94.3, 101.0)
- added XTRAPI_U2: W25Q128JVS, Package_SO:SOIC-8_5.23x5.23mm_P1.27mm, B.Cu at (88.0, 102.7)
- added XTRAPI_U3: RP2040, Package_DFN_QFN:QFN-56-1EP_7x7mm_P0.4mm_EP3.2x3.2mm, B.Cu at (86.4, 80.9)
- added XTRAPI_U4: AZ1117R-3_3TRE1, XTRAPI_JLC2KiCadLib:SOT-89-3_L4.5-W2.5-P1.50-LS4.2-BR, F.Cu at (88.7, 89.5)
- added XTRAPI_U6: B5819W_C8598, XTRAPI_JLC2KiCadLib:SOD-123_L2.7-W1.6-LS3.7-RD-1, F.Cu at (85.9, 95.8)
- added XTRAPI_U7: B5819W_C8598, XTRAPI_JLC2KiCadLib:SOD-123_L2.7-W1.6-LS3.7-RD-1, F.Cu at (88.9, 95.8)
- added XTRAPI_X1: X322512MSB4SI, XTRAPI_JLC2KiCadLib:OSC-SMD_4P-L3.2-W2.5-BL, B.Cu at (83.6, 74.3)
Routing:
- net GND: track 0.00 -> 474.3 mm, vias 0 -> 9
- net /XP_+3V3: track 0.00 -> 215.5 mm, vias 0 -> 5
- net VBUS: track 0.00 -> 215.0 mm, vias 0 -> 2
- net +3V3: track 0.00 -> 174.2 mm, vias 0 -> 8
- net /MOSFETOUT: track 0.00 -> 116.0 mm, vias 0 -> 3
- net /GPIO24: track 0.00 -> 91.6 mm, vias 0 -> 3
- net /ROW1: track 0.00 -> 88.7 mm, vias 0 -> 2
- net Net-(U3-USB_DP): track 0.00 -> 69.3 mm, vias 0 -> 1
- net Net-(J1-SHIELD): track 0.00 -> 66.6 mm, vias 0 -> 2
- net /MOSFETIN: track 0.00 -> 66.5 mm, vias 0 -> 3
- net /COL0: track 0.00 -> 63.2 mm, vias 0 -> 1
- net Net-(R9-Pad2): track 0.00 -> 63.2 mm, vias 0 -> 1
- net /XP_VBUS: track 0.00 -> 61.5 mm, vias 0 -> 4
- net Net-(U3-USB_DM): track 0.00 -> 58.0 mm, vias 0 -> 1
- net Net-(U8-A): track 0.00 -> 56.6 mm
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- added copper zone on B.Cu, net GND
- added copper zone on F.Cu, net GND
Other:
- board outline added: 90 x 100 mm
- board text added: "<- V-cut"
- board text added: "Powered by JLCPCB (https://jlcpcb.com/)"
- board text added: "T^3 The Teihen Tastatur - picopico"
- board text added: "with xtrapico"

Commit message: rel
Parts:
- added G2: LOGO, zeriparrot:zeriparrot, F.Cu at (97.4, 31.9)
- U10, U11, U12: value SK6812MINI-E_C5149201 -> RGBLED_SK6812MINI-E; footprint JLC2KiCadLib:LED-SMD_L3.2-W2.8-TR -> BrownSugar_KBD:RGBLED_SK6812MINI-E
- turned U10 to 0 degrees
- turned U11 to 0 degrees
- turned U12 to 0 degrees
Routing:
- net Net-(U10-DOUT): track 26.7 -> 35.4 mm, vias 0 -> 2
- net VBUS: track 215.0 -> 221.0 mm, vias 2 -> 6
- net /COL0: track 63.2 -> 65.3 mm, vias 1 -> 3
- net /RGBREV: track 35.8 -> 37.5 mm
- net /ROW0: track 37.4 -> 38.9 mm
- net /ROW1: track 88.7 -> 90.1 mm
- net Net-(U7-A): track 17.3 -> 15.9 mm, vias 0 -> 2
- net Net-(U13-+): track 32.0 -> 31.1 mm
- net Net-(U2-RUN): track 37.0 -> 37.9 mm
- net /ROT0IN: track 23.4 -> 24.3 mm
- net Net-(U11-DOUT): track 25.6 -> 25.1 mm
- net /MOSFETIN: track 66.5 -> 67.1 mm
Other:
- board text added: "BOOTSEL"
- board text added: "Powered by JLCPCB https://jlcpcb.com/"
- board text added: "RESET"
- board text added: "T^3 The Teihen Tastatur - picopico with xtrapico"
- board text removed: "Powered by JLCPCB (https://jlcpcb.com/)"
- board text removed: "T^3 The Teihen Tastatur - picopico"
- board text removed: "with xtrapico"
