File: picopico.kicad_sch (KiCad schematic)
At the start: 30 parts, among them J1 USB_C_Receptacle_USB2.0_14P, U1 1N4002W, U2 TD6810, U3 RP2040, X1 X322512MSB4SI

Commit message: rev1
Parts:
- added C10, C13: CL05A105KA5NQNC, JLC2KiCadLib:C0402, symbol CL05A105KA5NQNC:CL05A105KA5NQNC
- added C11, C12, C14, C15, C16, C17, C18, C19: CL05B104KO5NNNC, JLC2KiCadLib:C0402, symbol CL05B104KO5NNNC:CL05B104KO5NNNC
- added D1: WS2812B, LED_SMD:LED_WS2812B_PLCC4_5.0x5.0mm_P3.2mm, symbol LED:WS2812B
- added D2: LED, LED_SMD:LED_0402_1005Metric, symbol Device:LED
- added D3, D4, D5, D6: 0402ESDA-05N, JLC2KiCadLib:D0402-BI, symbol 0402ESDA-05N:0402ESDA-05N
- added J2: USB_C_Receptacle_USB2.0_14P, Connector_USB:USB_C_Receptacle_HRO_TYPE-C-31-M-12, symbol Connector:USB_C_Receptacle_USB2.0_14P
- added R12, R16, R17: 0402WGF1002TCE, JLC2KiCadLib:R0402, symbol 0402WGF1002TCE:0402WGF1002TCE
- added R13: 0603WAF2001T5E, JLC2KiCadLib:R0603, symbol 0603WAF2001T5E:0603WAF2001T5E
- added R14, R15: RC0402FR-0727RL, JLC2KiCadLib:R0402, symbol RC0402FR-0727RL:RC0402FR-0727RL
- added R18: 0402WGF4701TCE, JLC2KiCadLib:R0402, symbol 0402WGF4701TCE:0402WGF4701TCE
- added R19, R20: 0402WGF5101TCE, JLC2KiCadLib:R0402, symbol 0402WGF5101TCE:0402WGF5101TCE
- added SW1, SW2, SW3: SW_PUSH, PCM_Switch_Keyboard_Hotswap_Kailh:SW_Hotswap_Kailh_MX_1.00u, symbol BrownSugar_KBD:SW_PUSH
- added SW4: ~, BrownSugar_KBD:RotaryEncoder_EC11-Switch, symbol Device:RotaryEncoder_Switch
- added SW5, SW6: TSA343G00-250J2, JLC2KiCadLib:SW-SMD_L4.0-W2.9-LS5.0, symbol TSA343G00-250J2:TSA343G00-250J2
- added U10, U11, U12: SK6812MINI-E_C5149201, JLC2KiCadLib:LED-SMD_L3.2-W2.8-TR, symbol SK6812MINI-E_C5149201:SK6812MINI-E_C5149201
- added U13: FS-1540, JLC2KiCadLib:BUZ-SMD_5P-L15.0-W15.0-P13.7-BL, symbol FS-1540:FS-1540
- added U14, U4: X1321FR-2X20-C43D24, JLC2KiCadLib:CONN-TH_40P_X1321FR-2X20-C43D24, symbol X1321FR-2X20-C43D24:X1321FR-2X20-C43D24
- added U5, U6, U7, U8: 1N4148W_C81598, JLC2KiCadLib:SOD-123F_L2.7-W1.6-LS3.8-RD, symbol 1N4148W_C81598:1N4148W_C81598
- added U9: BSS138, JLC2KiCadLib:SOT-23-3_L2.9-W1.3-P1.90-LS2.4-BR, symbol BSS138:BSS138
- J1: footprint (none) -> Connector_USB:USB_C_Receptacle_HRO_TYPE-C-31-M-12
- renumbered SW_BOOTSEL2 to SW_RESET1
Connections:
- net +1V1: now also U3.23 (DVDD), U3.45 (VREG_VOUT), U3.50 (DVDD), C10.1, C11.1, C12.1
- net +3V3: now also U3.1 (IOVDD), U3.10 (IOVDD), U3.22 (IOVDD), U3.33 (IOVDD), U3.42 (IOVDD), U3.43 (ADC_AVDD), U3.44 (VREG_IN), U3.48 (USB_VDD), U3.49 (IOVDD), C13.1, C14.1, C15.1, C16.1, C17.1, C18.1, C19.1, R12.1, R16.1, U9.1 (G)
- net GND: now also C10.2, C11.2, C12.2, C13.2, C14.2, C15.2, C16.2, C17.2, C18.2, C19.2, D1.3 (VSS), D2.1 (K), D3.2, D4.2, D5.2, D6.2, J2.A1 (GND), J2.A12 (GND), J2.B1 (GND), J2.B12 (GND), R19.2, R20.2, SW4.C, SW5.2, SW6.2, U10.3 (GND), U11.3 (GND), U12.3 (GND), U13.2, U13.3, U13.4, U14.10, U14.12, U14.14, U14.6, U14.8, U4.14, U4.16, U4.18, U4.20, U4.22, U4.24, U4.26, U4.28, U4.30, U4.32, U4.34, U4.36
- net GPIO25: now also R18.1
- net VBUS: now also D1.1 (VDD), R17.2, U10.1 (VDD), U11.1 (VDD), U12.1 (VDD)
- net SWCLK: now reaches U3.24 (SWCLK)
- net SWCLK: now also U4.38
- net SWD: now reaches U3.25 (SWD)
- net SWD: now also U4.40
- net 3V3_EN: no longer names the net of R6.2, U2.1 (RUN)
- net GPIO0 renamed COL0
- net COL0: now also SW1.1, SW3.1
- net GPIO1 renamed COL1
- net COL1: now also SW2.1, SW4.S2
- net GPIO10: no longer names the net of U3.13 (GPIO10)
- net GPIO10: now also U4.7
- net GPIO11: no longer names the net of U3.14 (GPIO11)
- net GPIO11: now also U4.9
- net GPIO12: no longer names the net of U3.15 (GPIO12)
- net GPIO12: now also U4.11
- net GPIO13: no longer names the net of U3.16 (GPIO13)
- net GPIO13: now also U4.13
- net GPIO14: no longer names the net of U3.17 (GPIO14)
- net GPIO14: now also U4.15
- net GPIO15: no longer names the net of U3.18 (GPIO15)
- net GPIO15: now also U4.17
- net GPIO16: no longer names the net of U3.27 (GPIO16)
- net GPIO16: now also U4.19
- net GPIO17: no longer names the net of U3.28 (GPIO17)
- net GPIO17: now also U4.21
- net GPIO18: no longer names the net of U3.29 (GPIO18)
- net GPIO18: now also U4.23
- net GPIO19: no longer names the net of U3.30 (GPIO19)
- net GPIO19: now also U4.25
- net GPIO2 renamed ROW0
- net ROW0: now also U5.1 (K), U6.1 (K)
- net GPIO20: no longer names the net of U3.31 (GPIO20)
- net GPIO20: now also U4.27
- net GPIO21: no longer names the net of U3.32 (GPIO21)
- net GPIO21: now also U4.29
- net GPIO22: no longer names the net of U3.34 (GPIO22)
- net GPIO22: now also U4.31
- net GPIO23: no longer names the net of U3.35 (GPIO23)
- net GPIO23: now also U4.33
- net GPIO26_ADC0: no longer names the net of U3.38 (GPIO26_ADC0)
- net GPIO26_ADC0: now also U4.35
- net GPIO27_ADC1: no longer names the net of U3.39 (GPIO27_ADC1)
- net GPIO27_ADC1: now also U4.37
- net GPIO28_ADC2: no longer names the net of U3.40 (GPIO28_ADC2)
- net GPIO28_ADC2: now also U4.39
- net GPIO29_ADC3: no longer names the net of U3.41 (GPIO29_ADC3)
- net GPIO29_ADC3: now also U13.1 (+)
- net GPIO3 renamed ROW1
- net ROW1: now also U7.1 (K), U8.1 (K)
- net GPIO4 renamed ROT0IN
- net ROT0IN: now also SW4.B
- net GPIO5 renamed ROT0OUT
- net ROT0OUT: now also SW4.A
- net GPIO6 renamed RGBEXT
- net RGBEXT: now also U4.2
- net GPIO7: no longer names the net of U3.9 (GPIO7)
- net GPIO7: now also U4.1
- net GPIO8: no longer names the net of U3.11 (GPIO8)
- net GPIO8: now also U4.3
- net GPIO9: no longer names the net of U3.12 (GPIO9)
- net GPIO9: now also U4.5
- net USB_DN: no longer names the net of J1.A7 (D-), J1.B7 (D-)
- net USB_DN: now also R15.1; no longer U3.46 (USB_DM)
- net USB_DP: no longer names the net of J1.A6 (D+), J1.B6 (D+)
- net USB_DP: now also R14.1; no longer U3.47 (USB_DP)
- new net: J2.A5 (CC1), R20.1
- new net: J2.B5 (CC2), R19.1
- new net: U11.2 (DOUT), U12.4 (DIN)
- new net: U10.2 (DOUT), U11.4 (DIN)
- new net: R12.2, R13.1
- new net: SW4.S1, U8.2 (A)
- new net: SW2.2, U6.2 (A)
- new net: R14.2, U3.47 (USB_DP)
- new net: SW1.2, U5.2 (A)
- new net: SW3.2, U7.2 (A)
- new net: D2.2 (A), R18.2
- new net: R15.2, U3.46 (USB_DM)
- new net +3.3V: R13.2
- new net MOSFETIN: R16.2, U4.8, U9.2 (S)
- new net MOSFETOUT: R17.1, U4.10, U9.3 (D)
- new net RGBREV: U10.4 (DIN), U4.12
- new net WSIN: D1.4 (DIN), U4.4
- new net WSOUT: D1.2 (DOUT), U4.6
- new net XP_+3V3: U14.18
- new net XP_BOOTSEL: SW6.1
- new net XP_GPIO0: U14.1
- new net XP_GPIO1: U14.3
- new net XP_GPIO10: U14.21
- new net XP_GPIO11: U14.23
- new net XP_GPIO12: U14.25
- new net XP_GPIO13: U14.27
- new net XP_GPIO14: U14.29
- new net XP_GPIO15: U14.31
- new net XP_GPIO16: U14.33
- new net XP_GPIO17: U14.35
- new net XP_GPIO18: U14.37
- new net XP_GPIO19: U14.39
- new net XP_GPIO2: U14.5
- new net XP_GPIO20: U14.40
- new net XP_GPIO21: U14.38
- new net XP_GPIO22: U14.36
- new net XP_GPIO23: U14.34
- new net XP_GPIO24: U14.32
- new net XP_GPIO25: U14.30
- new net XP_GPIO26_ADC0: U14.28
- new net XP_GPIO27_ADC1: U14.26
- new net XP_GPIO28_ADC2: U14.24
- new net XP_GPIO29_ADC3: U14.22
- new net XP_GPIO3: U14.7
- new net XP_GPIO4: U14.9
- new net XP_GPIO5: U14.11
- new net XP_GPIO6: U14.13
- new net XP_GPIO7: U14.15
- new net XP_GPIO8: U14.17
- new net XP_GPIO9: U14.19
- new net XP_RUN: SW5.1
- new net XP_SWCLK: U14.2
- new net XP_SWD: U14.4
- new net XP_USB_DN: D6.1, J2.A7 (D-), J2.B7 (D-)
- new net XP_USB_DP: D5.1, J2.A6 (D+), J2.B6 (D+)
- new net XP_VBUS: D3.1, D4.1, J2.A4 (VBUS), J2.A9 (VBUS), J2.B4 (VBUS), J2.B9 (VBUS), U14.20
- new net XP_VSYS: U14.16
- no-connect marks 4 -> 6
Other:
- added sheet xtrapico core (third_party/zeriyoshi/xtrapico/core.kicad_sch)
- moved on the sheet: C7

Commit message: rel
Parts:
- removed U10, U11, U12: SK6812MINI-E_C5149201, JLC2KiCadLib:LED-SMD_L3.2-W2.8-TR, symbol SK6812MINI-E_C5149201:SK6812MINI-E_C5149201
- added U10, U11, U12: RGBLED_SK6812MINI-E, BrownSugar_KBD:RGBLED_SK6812MINI-E, symbol BrownSugar_KBD:RGBLED_SK6812MINI-E
Connections:
- net GND: now also U10.3 (GND), U11.3 (GND), U12.3 (GND)
- net RGBREV: now also U10.4 (DIN)
- net VBUS: now also U10.1 (VDD), U11.1 (VDD), U12.1 (VDD)
- new net: U11.2 (DOUT), U12.4 (DIN)
- new net: U10.2 (DOUT), U11.4 (DIN)
